File: Power.kicad_sch (KiCad schematic)
At the start: 5 parts, among them U1 INA237, U2 MIC5504-3.3YM5-TR

Commit message: fixed stuff
Parts:
- added D1: D, Diode_THT:D_DO-35_SOD27_P7.62mm_Horizontal, symbol Device:D
- added F1: Polyfuse, Package_LCC:PLCC-84_29.3x29.3mm_P1.27mm, symbol Device:Polyfuse
- VIN: renamed from 5V; value GND -> PWR_IN; footprint (none) -> TerminalBlock:TerminalBlock_MaiXu_MX126-5.0-02P_1x02_P5.00mm
Connections:
- net 5V: now also D1.1 (K); no longer VIN.1 (Pin_1)
- net GND: no longer VIN.2 (Pin_2)
- new net: D1.2 (A), F1.2
- new net: F1.1, VIN.1 (Pin_1)
Other:
- moved on the sheet: R1, VIN

Commit message: more fixes
Parts:
- added C15: 100nF, symbol Device:C
- added C16: 1uF, symbol Device:C
- added J4: Screw_Terminal_01x02, TerminalBlock:TerminalBlock_MaiXu_MX126-5.0-02P_1x02_P5.00mm, symbol Connector:Screw_Terminal_01x02
- C1: value C -> 10 uF; footprint rov_power:SOT-23-5_MC_MCH -> Capacitor_SMD:C_0201_0603Metric
- U1: footprint Package_SO:TSSOP-10_3x3mm_P0.5mm -> rov_sensors:VSSOP_IDGSR_TEX
Connections:
- net 3V3: now also C15.1, C16.1
- net GND: now also C15.2, C16.2, J4.2 (Pin_2)
- net 5V renamed 5V_IN
- net 5V_IN: now also U2.1 (VIN), U2.3 (EN); no longer U1.8 (Vbus)
- net POST_SHUNT renamed 5V_PI
- net 5V_PI: now also U1.8 (Vbus), J4.1 (Pin_1); no longer U2.1 (VIN), U2.3 (EN)
Other:
- moved on the sheet: C1, R1, U1

Commit message: i did stuff
Parts:
- added D2: LED, symbol Device:LED
- added J9: TEST_PWR, TerminalBlock_4Ucon:TerminalBlock_4Ucon_1x02_P3.50mm_Vertical, symbol Connector:Screw_Terminal_01x02
- added R6: 330, symbol Device:R
- added TP1, TP2: TestPoint, TestPoint:TestPoint_Loop_D2.50mm_Drill1.0mm_LowProfile, symbol Connector:TestPoint
- renumbered C15 to C2, C16 to C3, J4 to J1, U2 to U1, U1 to U2, VIN to VIN1
Connections:
- net 3V3: now also R6.2, TP1.1
- net 5V_IN: now also TP2.1
- net GND: now also VIN1.2 (Pin_2), D2.2 (A), J9.2 (Pin_2)
- net at F1.1, VIN1.1 (Pin_1): now also J9.1 (Pin_1)
- new net: D2.1 (K), R6.1
- no-connect marks 0 -> 1
Other:
- moved on the sheet: C1, D1, F1
