File: Sensor.kicad_sch (KiCad schematic)
At the start: 6 parts, among them U4 BME280, U5 TMP1075NDRLR, U6 BNO085, U7 BMI270

Commit message: fixed stuff
Changed lines of the file:
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@@
 	)
 	(global_label "SCL"
-		(shape input)
+		(shape bidirectional)
 		(at 163.83 59.69 180)
 		(fields_autoplaced yes)
@@
 		)
 		(property "Intersheetrefs" "${INTERSHEET_REFS}"
-			(at 157.3372 59.69 0)
+			(at 156.2259 59.69 0)
 			(hide yes)
 			(show_name no)
@@
 	)
 	(global_label "SDA"
-		(shape input)
+		(shape bidirectional)
 		(at 204.47 59.69 0)
 		(fields_autoplaced yes)
@@
 		)
 		(property "Intersheetrefs" "${INTERSHEET_REFS}"
-			(at 211.0233 59.69 0)
+			(at 212.1346 59.69 0)
 			(hide yes)
 			(show_name no)
@@
 	)
 	(global_label "SCL"
-		(shape input)
+		(shape bidirectional)
 		(at 223.52 83.82 0)
 		(fields_autoplaced yes)
@@
 		)
 		(property "Intersheetrefs" "${INTERSHEET_REFS}"
-			(at 230.0128 83.82 0)
+			(at 231.1241 83.82 0)
 			(hide yes)
 			(show_name no)
@@
 	)
 	(global_label "SCL"
-		(shape input)
+		(shape bidirectional)
 		(at 133.35 114.3 0)
 		(fields_autoplaced yes)
@@
 		)
 		(property "Intersheetrefs" "${INTERSHEET_REFS}"
-			(at 139.8428 114.3 0)
+			(at 140.9541 114.3 0)
 			(hide yes)
 			(show_name no)
@@
 	)
 	(global_label "SDA"
-		(shape input)
+		(shape bidirectional)
 		(at 242.57 128.27 0)
 		(fields_autoplaced yes)
@@
 		)
 		(property "Intersheetrefs" "${INTERSHEET_REFS}"
-			(at 249.1233 128.27 0)
+			(at 250.2346 128.27 0)
 			(hide yes)
 			(show_name no)
@@
 	)
 	(global_label "SCL"
-		(shape input)
+		(shape bidirectional)
 		(at 135.89 63.5 0)
 		(fields_autoplaced yes)
@@
 		)
 		(property "Intersheetrefs" "${INTERSHEET_REFS}"
-			(at 142.3828 63.5 0)
+			(at 143.4941 63.5 0)
 			(hide yes)
 			(show_name no)
@@
 	)
 	(global_label "SDA"
-		(shape input)
+		(shape bidirectional)
 		(at 133.35 111.76 0)
 		(fields_autoplaced yes)
@@
 		)
 		(property "Intersheetrefs" "${INTERSHEET_REFS}"
-			(at 139.9033 111.76 0)
+			(at 141.0146 111.76 0)
 			(hide yes)
 			(show_name no)
@@
 	)
 	(global_label "SCL"
-		(shape input)
+		(shape bidirectional)
 		(at 242.57 130.81 0)
 		(fields_autoplaced yes)
@@
 		)
 		(property "Intersheetrefs" "${INTERSHEET_REFS}"
-			(at 249.0628 130.81 0)
+			(at 250.1741 130.81 0)
 			(hide yes)
 			(show_name no)
@@
 	)
 	(global_label "SDA"
-		(shape input)
+		(shape bidirectional)
 		(at 232.41 83.82 0)
 		(fields_autoplaced yes)
@@
 		)
 		(property "Intersheetrefs" "${INTERSHEET_REFS}"
-			(at 238.9633 83.82 0)
+			(at 240.0746 83.82 0)
 			(hide yes)
 			(show_name no)
@@
 	)
 	(global_label "SDA"
-		(shape input)
+		(shape bidirectional)
 		(at 135.89 68.58 0)
 		(fields_autoplaced yes)
@@
 		)
 		(property "Intersheetrefs" "${INTERSHEET_REFS}"
-			(at 142.4433 68.58 0)
-			(hide yes)
-			(show_name no)
+			(at 143.5546 68.58 0)
+			(hide yes)
+			(show_name no)

Commit message: more fixes
Parts:
- added C18, C19, C20, C21, C22, C23, C24, C25: 100nF, symbol Device:C
- R2, R3: footprint rov_sensors:Bosch_LGA-14_3x2.5mm_P0.5mm -> Resistor_SMD:R_0201_0603Metric
Connections:
- net 3V3: now also U6.10 (CLKSEL0), C19.1, C20.1, C21.1, C23.1, C24.1, C25.1; no longer U6.11 (NRST)
- net GND: now also U6.24 (RESV_NC), C18.2, C19.2, C20.2, C21.2, C22.2, C23.2, C24.2, C25.2
- net BNO_INT: now reaches U6.14 (H_INTN)
- net at U6.9 (CAP): now also C18.1
- new net BNO_RST: U6.11 (NRST)
- no-connect marks 0 -> 6

Commit message: i did stuff
Parts:
- renumbered C25 to C10, C20 to C11, C21 to C4, C23 to C5, C24 to C6, C22 to C7, C18 to C8, C19 to C9, R3 to R2, R2 to R3, U7 to U3
Connections:
- net 3V3: now also C7.1
- no-connect marks 6 -> 11
Other:
- moved on the sheet: C7
