File: X-19-Testbench-Sensor-Pi.kicad_sch (KiCad schematic)
At the start: 0 parts

Commit message: i did stuff
Other:
- sheet CAN ports: added 3V3, 5V_IN, CAN_RX, CAN_TX, MCP_CS, MCP_IN, MISO, MOSI, SCK; removed none
- sheet Compute ports: added 3V3, BNO_INT, BNO_RST, CAN_RX, CAN_TX, MCP_CS, MCP_IN, MISO, MOSI, SCK, SCL, SDA; removed none
- sheet Power ports: added 3V3, 5V_IN, SCL, SDA; removed none
- sheet Sensor ports: added 3V3, BNO_INT, BNO_RST, SCL, SDA; removed none
